Commit message: robot arm urdf modification

File: urdf/robot_arm (copy).urdf (robot description, URDF)
Before this commit: robot robot_arm, 9 links, 8 joints
Links:
- link base_link: geometry collision box size=0.2 0.2 0.7; visual box size=0.2 0.2 1
- link base_link_p: geometry collision box size=1 1 0.2; visual box size=1 1 0.2
- link box: geometry collision box size=1 1 0.2; visual box size=1 1 0.2
- link link1_p: geometry collision box size=1 1 0.2; visual box size=1 1 0.2
- link link3: geometry collision cylinder length=1 radius=0.1; visual cylinder length=1 radius=0.1
- link link4: geometry collision cylinder length=0.4 radius=0.07; visual cylinder length=0.4 radius=0.07
Joints:
- joint joint1: origin xyz=0 0 1.2 rpy=0 0 0 -> xyz=0 0 1 rpy=0 0 0
- joint joint4: origin xyz=0 0 0.3 rpy=0 0 0 -> xyz=0 0 1 rpy=0 0 0
- joint joint5: origin xyz=0 1.5 0.25 rpy=0 0 0 -> xyz=0 2.5 0.25 rpy=0 0 0
