Commit message: robot arm and rotational platform

File: urdf/robot_arm.urdf (robot description, URDF)
Before this commit: robot gripper_robot, 6 links, 5 joints
Links:
- added link base_link_p, mass 1; collision box size=1 1 0.2; visual box size=1 1 0.2
- added link link1_p, mass 1; collision box size=1 1 0.2; visual box size=1 1 0.2
Joints:
- added joint joint5: type revolute, parent base_link_p, child link1_p, origin xyz=0 2.5 0.25 rpy=0 0 0, axis 0 0 1, limit lower=-1.5708 upper=1.5708 effort=100 velocity=100
- added joint joint_fix_p: type fixed, parent world, child base_link_p

Commit message: version1

File: urdf/robot_arm.urdf (robot description, URDF)
Before this commit: robot robot_arm, 9 links, 8 joints
Links:
- link base_link: geometry collision box size=0.2 0.2 1.5; visual box size=0.2 0.2 1.8
- link link2: geometry collision cylinder length=1.1 radius=0.09; visual cylinder length=1.2 radius=0.09
- link link3: geometry collision cylinder length=0.3 radius=0.07; visual cylinder length=0.3 radius=0.07
Joints:
- joint joint1: origin xyz=0 0 1.2 rpy=0 0 0 -> xyz=0 0 1.5 rpy=0 0 0
- joint joint3: origin xyz=0 0 1 rpy=0 0 0 -> xyz=0 0 1.2 rpy=0 0 0
- joint joint5: limit lower=-1.5708 upper=1.5708 effort=100 velocity=100 -> lower=-3.1416 upper=3.1416 effort=100 velocity=100; origin xyz=0 1.5 0.25 rpy=0 0 0 -> xyz=0 1.5 0.15 rpy=0 0 0

Commit message: satisfied demo

File: urdf/robot_arm.urdf (robot description, URDF)
Before this commit: robot robot_arm, 9 links, 8 joints
Links:
- link base_link: geometry collision box size=0.2 0.2 1.4; visual box size=0.2 0.2 1.6
- link box: geometry collision box size=0.45 0.36 0.78; visual box size=0.45 0.36 0.78
- link link1: geometry collision cylinder length=0.1 radius=0.09; visual cylinder length=0.1 radius=0.09
- link link1_p: geometry collision cylinder length=0.1 radius=0.75; visual cylinder length=0.1 radius=0.75
- link link2: geometry collision cylinder length=1.1 radius=0.07; visual cylinder length=1.2 radius=0.07
- link link3: geometry collision cylinder length=0.3 radius=0.04; visual cylinder length=0.3 radius=0.04
- link link4: geometry collision cylinder length=0.12 radius=0.025; visual cylinder length=0.12 radius=0.025
Joints:
- joint joint1: limit lower=-1.5708 upper=1.5708 effort=100 velocity=100 -> lower=0 upper=3.1416 effort=100 velocity=100
