Commit message: joint fixed

File: urdf/robot_demo.urdf (robot description, URDF)
Before this commit: robot robot_demo, 7 links, 6 joints
Joints:
- removed joint joint
- added joint joint1: type fixed, parent base_link, child link1, origin xyz=0 0 0.11 rpy=1.5707963267949 0 0, axis 0 1 0
- joint joint_camera: axis 0 0 1 -> 0 0 0

Commit message: robot_demo

File: urdf/robot_demo.urdf (robot description, URDF)
Before this commit: robot demo_test, 3 links, 2 joints
Links:
- removed link world
- added link camera, mass 0.430020999525805; collision mesh filename=package://robot_demo/meshes/camera.STL; visual mesh filename=package://robot_demo/meshes/camera.STL
- added link link2, mass 28.7296694386766; collision mesh filename=package://robot_demo/meshes/link2.STL; visual mesh filename=package://robot_demo/meshes/link2.STL
- added link link3, mass 16.0188527649003; collision mesh filename=package://robot_demo/meshes/link3.STL; visual mesh filename=package://robot_demo/meshes/link3.STL
- added link link4, mass 2.22702219995936; collision mesh filename=package://robot_demo/meshes/link4.STL; visual mesh filename=package://robot_demo/meshes/link4.STL
- added link link5, mass 0.844952599159698; collision mesh filename=package://robot_demo/meshes/link5.STL; visual mesh filename=package://robot_demo/meshes/link5.STL
- link base_link: geometry collision mesh filename=package://robot_demo/meshes/base_link.STL; visual mesh filename=package://robot_demo/meshes/base_link.STL
- link link1: geometry collision mesh filename=package://robot_demo/meshes/link1.STL; visual mesh filename=package://robot_demo/meshes/link1.STL
Joints:
- removed joint joint_fix
- added joint joint2: type continuous, parent link1, child link2, origin xyz=0 0.322732802998902 -0.250383739680009 rpy=0 0 0, axis 1 0 0
- added joint joint3: type continuous, parent link2, child link3, origin xyz=0 1.13860941000177 0 rpy=0 0 0, axis 1 0 0
- added joint joint4: type continuous, parent link5, child link4, origin xyz=0 0 0 rpy=0 0 0, axis 1 0 0
- added joint joint5: type continuous, parent link3, child link5, origin xyz=0.0483407685108505 0 -0.693420367397096 rpy=0 0 0, axis 0 1 0
- added joint joint_camera: type fixed, parent link4, child camera, origin xyz=0 0 -0.18 rpy=0 0 0, axis 0 0 0
- joint joint1: limit lower=0 upper=3.1416 effort=100 velocity=100 -> (none); origin xyz=0 -1.5 0.11 rpy=1.5707963267949 0 0 -> xyz=0 0 0.11 rpy=1.5707963267949 0 0; type revolute -> fixed
