Commit message: whole

File: urdf/demo.urdf (robot description, URDF)
Before this commit: robot demo, 7 links, 6 joints
Links:
- added link world
- link base_link: geometry collision mesh filename=package://demo_test/meshes/base_link.STL; visual mesh filename=package://demo_test/meshes/base_link.STL
- link base_rot: geometry collision mesh filename=package://demo_test/meshes/base_rot.STL; visual mesh filename=package://demo_test/meshes/base_rot.STL
- link link1: geometry collision mesh filename=package://demo_test/meshes/link1.STL; visual mesh filename=package://demo_test/meshes/link1.STL
- link link2: geometry collision mesh filename=package://demo_test/meshes/link2.STL; visual mesh filename=package://demo_test/meshes/link2.STL
- link link3: geometry collision mesh filename=package://demo_test/meshes/link3.STL; visual mesh filename=package://demo_test/meshes/link3.STL
- link link4: geometry collision mesh filename=package://demo_test/meshes/link4.STL; visual mesh filename=package://demo_test/meshes/link4.STL
- link plate: geometry collision mesh filename=package://demo_test/meshes/plate.STL; visual mesh filename=package://demo_test/meshes/plate.STL
Joints:
- added joint joint_fix: type fixed, parent world, child base_link
- joint joint1: limit (none) -> lower=0 upper=3.1416 effort=100 velocity=100; type continuous -> revolute
- joint joint2: limit (none) -> lower=0 upper=3.1416 effort=100 velocity=100; type continuous -> revolute
- joint joint3: limit (none) -> lower=0 upper=3.1416 effort=100 velocity=100; type continuous -> revolute
- joint joint4: limit (none) -> lower=0 upper=3.1416 effort=100 velocity=100; type continuous -> revolute
- joint joint5: limit (none) -> lower=0 upper=3.1416 effort=100 velocity=100; type continuous -> revolute
- joint joint_p: parent base_link -> world

Commit message: demo

File: urdf/demo.urdf (robot description, URDF)
Before this commit: robot demo, 8 links, 7 joints
Joints:
- joint joint1: origin xyz=0 -1.5 0.11 rpy=1.5707963267949 0 0 -> xyz=0 0 0.11 rpy=1.5707963267949 0 0

File: urdf/robot_demo.urdf (robot description, URDF)
Before this commit: robot robot_demo, 7 links, 6 joints
Links:
- removed link camera
- removed link link2
- removed link link3
- removed link link4
- removed link link5
- added link world
- link base_link: geometry collision mesh filename=package://demo_test/meshes/base_link.STL; visual mesh filename=package://demo_test/meshes/base_link.STL
- link link1: geometry collision mesh filename=package://demo_test/meshes/link1.STL; visual mesh filename=package://demo_test/meshes/link1.STL
Joints:
- removed joint joint2
- removed joint joint3
- removed joint joint4
- removed joint joint5
- removed joint joint_camera
- added joint joint_fix: type fixed, parent world, child base_link
- joint joint1: limit (none) -> lower=0 upper=3.1416 effort=100 velocity=100; origin xyz=0 0 0.11 rpy=1.5707963267949 0 0 -> xyz=0 -1.5 0.11 rpy=1.5707963267949 0 0; type fixed -> revolute

Commit message: frame

File: urdf/demo.urdf (robot description, URDF)
Before this commit: robot demo, 8 links, 7 joints
Links:
- removed link base_rot
- removed link plate
- added link link5, mass 0.844952599159698; visual mesh filename=package://demo_test/meshes/link5.STL
- link link4: geometry visual mesh filename=package://demo_test/meshes/link4.STL
Joints:
- removed joint joint_p
- joint joint3: origin xyz=0 0.84737046476322 0 rpy=0 0 0 -> xyz=0 1.13860941000177 0 rpy=0 0 0
- joint joint4: origin xyz=0.0383407685108506 0 -0.603280829801762 rpy=0 0 -1.5707963267949 -> xyz=0.0383407685108506 0 0 rpy=0 0 0; parent link3 -> link5
- joint joint5: child plate -> link5; limit lower=0 upper=3.1416 effort=100 velocity=100 -> (none); origin xyz=0 0.15 0 rpy=0 0 0 -> xyz=0.0483407685108505 0 -0.693420367397096 rpy=0 0 0; parent base_rot -> link3; type revolute -> continuous

Commit message: 15

File: urdf/demo.urdf (robot description, URDF)
Before this commit: robot demo, 7 links, 6 joints
Links:
- added link camera, mass 0.430020999525805; visual mesh filename=package://robot_demo/meshes/camera.STL
- link base_link: geometry visual mesh filename=package://demo_test/meshes/base_link.STL
- link link1: geometry visual mesh filename=package://demo_test/meshes/link1.STL
- link link2: geometry visual mesh filename=package://demo_test/meshes/link2.STL
- link link3: geometry visual mesh filename=package://demo_test/meshes/link3.STL
Joints:
- added joint joint_camera: type fixed, parent link4, child camera, origin xyz=0 0 -0.18 rpy=0 0 0, axis 0 0 0

Commit message: model done

File: urdf/demo.urdf (robot description, URDF)
Before this commit: robot demo, 8 links, 7 joints
Links:
- added link base_link_p, mass 1; collision box size=1 1 0.1; visual box size=1 1 0.1
- added link box, mass 1; collision box size=0.45 0.36 0.78; visual box size=0.45 0.36 0.78
- added link link1_p, mass 1; collision cylinder length=0.1 radius=0.75; visual cylinder length=0.1 radius=0.75
- link camera: geometry visual mesh filename=package://demo_test/meshes/camera.STL
Joints:
- added joint joint6: type revolute, parent base_link_p, child link1_p, origin xyz=0 1.5 0.15 rpy=0 0 0, axis 0 0 1, limit lower=-3.1416 upper=3.1416 effort=100 velocity=100
- added joint joint_box: type fixed, parent link1_p, child box
- added joint joint_fix_p: type fixed, parent world, child base_link_p
- joint joint4: origin xyz=0.0383407685108506 0 0 rpy=0 0 0 -> xyz=0 0 0 rpy=0 0 0
- joint joint_camera: limit (none) -> lower=0 upper=3.1416 effort=100 velocity=100; type fixed -> revolute

Commit message: jiben

File: urdf/demo.urdf (robot description, URDF)
Before this commit: robot demo, 11 links, 10 joints
Links:
- link box: geometry collision mesh filename=package://demo_test/meshes/frig.STL; visual mesh filename=package://demo_test/meshes/frig.STL
Joints:
- removed joint joint_camera
- added joint joint7: type revolute, parent base_link_p, child link1_p, origin xyz=0 2.5 0.15 rpy=0 0 0, axis 0 0 1, limit lower=-3.1416 upper=3.1416 effort=100 velocity=100
- joint joint1: limit lower=0 upper=3.1416 effort=100 velocity=100 -> lower=-3.1416 upper=3.1416 effort=100 velocity=100
- joint joint2: limit lower=0 upper=3.1416 effort=100 velocity=100 -> lower=-3.1416 upper=3.1416 effort=100 velocity=100
- joint joint3: limit lower=0 upper=3.1416 effort=100 velocity=100 -> lower=-3.1416 upper=3.1416 effort=100 velocity=100
- joint joint4: axis -1 0 0 -> 0 1 0; child link4 -> link5; limit lower=0 upper=3.1416 effort=100 velocity=100 -> lower=-3.1416 upper=3.1416 effort=100 velocity=100; origin xyz=0 0 0 rpy=0 0 0 -> xyz=0.0483407685108505 0 -0.693420367397096 rpy=0 0 0; parent link5 -> link3
- joint joint5: axis 0 1 0 -> -1 0 0; child link5 -> link4; limit (none) -> lower=-3.1416 upper=3.1416 effort=100 velocity=100; origin xyz=0.0483407685108505 0 -0.693420367397096 rpy=0 0 0 -> xyz=0 0 0 rpy=0 0 0; parent link3 -> link5; type continuous -> revolute
- joint joint6: axis 0 0 1 -> 0 0 0; child link1_p -> camera; origin xyz=0 1.5 0.15 rpy=0 0 0 -> xyz=0 0 -0.18 rpy=0 0 0; parent base_link_p -> link4

Commit message: haixing

File: urdf/demo.urdf (robot description, URDF)
Before this commit: robot demo, 11 links, 10 joints
Links:
- link base_link: mass 17.8923575005348 -> 0.1
- link link1: mass 19.3943177662416 -> 0.1
- link link2: mass 22.5828591680831 -> 0.1
- link link3: mass 13.649633544176 -> 0.1
- link link4: mass 3.83524054978555 -> 0.1
- link link5: mass 0.844952599159698 -> 0.1
Joints:
- joint joint7: origin xyz=0 2.5 0.15 rpy=0 0 0 -> xyz=0 2.0 0.15 rpy=0 0 0

Commit message: fff

File: urdf/demo.urdf (robot description, URDF)
Before this commit: robot demo, 11 links, 10 joints
Links:
- link camera: mass 0.430020999525805 -> 0.001
- link link2: mass 0.1 -> 5
- link link4: mass 0.1 -> 0.001
- link link5: mass 0.1 -> 0.01
